File: Proyecto de KiCad/TPFinal_Embebidos/TPFinal_Embebidos.kicad_pcb (KiCad board)
At the start: 2 copper layers, 130 x 150 mm, 13 parts, among them CN10 Conn_02x19_Odd_Even, CN7 Conn_02x19_Odd_Even, U2 LM35

Commit message: Add files via upload
Routing:
- net +5V: track 293.1 -> 336.6 mm
- net GND: track 342.6 -> 376.4 mm
Changed lines of the file:
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@@
+	)
+	(segment
+		(start 202.208 57.912)
+		(end 209.55 57.912)
+		(width 1)
+		(layer "B.Cu")
+		(net 8)
 	)
 	(segment
@@
 	)
 	(segment
+		(start 191.77 42.926)
+		(end 192.786 43.942)
+		(width 1)
+		(layer "B.Cu")
+		(net 8)
+	)
+	(segment
 		(start 199.208 150.296)
 		(end 232.006 150.296)
@@
 	)
 	(segment
+		(start 187.706 46.99)
+		(end 187.706 44.704)
+		(width 1)
+		(layer "B.Cu")
+		(net 8)
+	)
+	(segment
+		(start 192.786 48.49)
+		(end 202.208 57.912)
+		(width 1)
+		(layer "B.Cu")
+		(net 8)
+	)
+	(segment
+		(start 192.786 46.99)
+		(end 192.786 48.49)
+		(width 1)
+		(layer "B.Cu")
+		(net 8)
+	)
+	(segment
 		(start 224.79 57.912)
-		(end 208.788 57.912)
+		(end 209.55 57.912)
+		(width 1)
+		(layer "B.Cu")
+		(net 8)
+	)
+	(segment
+		(start 189.484 42.926)
+		(end 191.77 42.926)
+		(width 1)
+		(layer "B.Cu")
+		(net 8)
+	)
+	(segment
+		(start 187.706 44.704)
+		(end 189.484 42.926)
 		(width 1)
 		(layer "B.Cu")
@@
 	)
 	(segment
+		(start 209.55 57.912)
+		(end 208.788 57.912)
+		(width 1)
+		(layer "B.Cu")
+		(net 8)
+	)
+	(segment
 		(start 238.76 140.462)
 		(end 238.962 140.26)
@@
 	)
 	(segment
+		(start 192.786 43.942)
+		(end 192.786 46.99)
+		(width 1)
+		(layer "B.Cu")
+		(net 8)
+	)
+	(segment
 		(start 244.348 131.318)
 		(end 244.348 140.716)
@@
 	)
 	(segment
+		(start 195.326 38.1)
+		(end 192.024 34.798)
+		(width 1)
+		(layer "B.Cu")
+		(net 17)
+	)
+	(segment
+		(start 195.326 46.99)
+		(end 195.326 38.1)
+		(width 1)
+		(layer "B.Cu")
+		(net 17)
+	)
+	(segment
 		(start 222.758 83.82)
 		(end 126.165 83.82)
@@
 		(width 1)
 		(layer "B.Cu")
+		(net 17)
+	)
+	(segment
+		(start 192.024 34.798)
+		(end 162.052 34.798)
+		(width 1)
+		(layer "B.Cu")
